File: KiCad/MicSparkCal/MicSparkCal.kicad_pcb (KiCad board)
At the start: 2 copper layers, 88 x 55 mm, 36 parts, among them J1 Cortex Debug, J10 TF_S_A, J11 TF_S_B, J12 HV_A, J13 HV_B, J2 ON/OFF, J3 BOOST_IN_P, J4 BOOST_IN_N, J5 BOOST_OUT_P, J6 BOOST_OUT_N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

Commit message: Set h/w revision to 2 and include some fixes
Parts:
- removed J6: BOOST_OUT_N, Connector_PinHeader_2.54mm:PinHeader_1x01_P2.54mm_Vertical
- J4: value BOOST_IN_N -> BOOST_COMM
Routing:
- net +12V: track 82.2 -> 91.1 mm, vias 1 -> 2
- net GNDPWR: vias 65 -> 66
